File: Electronics/3x4-12-key-numpad.sch (KiCad schematic (older format))
At the start: 35 parts, among them J1 USB_mini_micro_B, K1 KEYSW, K10 KEYSW, K11 KEYSW, K12 KEYSW, K2 KEYSW, K3 KEYSW, K4 KEYSW, K5 KEYSW, K6 KEYSW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

Commit message: Added images
Parts:
- added D13: LED_ALT, LEDs:LED_0805_HandSoldering, symbol LED_ALT
- added R5: 10k, Resistors_SMD:R_0805_HandSoldering, symbol R
- renumbered C8 to C3
Connections:
- net GND: now also R5.2
- net at U1.14 (PB0): now also D13.2 (A)
- new net: D13.1 (K), R5.1
- no-connect marks 13 -> 12
Other:
- note added: "1"
- note added: "Shuttle\n"
Changed lines of the file:
@@
 EELAYER 25 0
 EELAYER END
-$Descr A4 11693 8268
+$Descr User 8661 5906
 encoding utf-8
 Sheet 1 1
@@
 $EndComp
 $Comp
-L VCC #PWR04
+L VCC #PWR02
 U 1 1 59DD1624
 P 6350 1400
-F 0 "#PWR04" H 6350 1250 50  0001 C CNN
+F 0 "#PWR02" H 6350 1250 50  0001 C CNN
 F 1 "VCC" H 6350 1550 50  0000 C CNN
 F 2 "" H 6350 1400 50  0001 C CNN
@@
 $EndComp
 $Comp
-L GND #PWR05
+L GND #PWR03
 U 1 1 59DD164E
 P 6350 1650
-F 0 "#PWR05" H 6350 1400 50  0001 C CNN
+F 0 "#PWR03" H 6350 1400 50  0001 C CNN
 F 1 "GND" H 6350 1500 50  0000 C CNN
 F 2 "" H 6350 1650 50  0001 C CNN
@@
 $EndComp
 $Comp
-L GND #PWR06
+L GND #PWR04
 U 1 1 59DD1F34
 P 2550 2050
-F 0 "#PWR06" H 2550 1800 50  0001 C CNN
+F 0 "#PWR04" H 2550 1800 50  0001 C CNN
 F 1 "GND" H 2550 1900 50  0000 C CNN
 F 2 "" H 2550 2050 50  0001 C CNN
@@
 $EndComp
 $Comp
-L C C8
+L C C3
 U 1 1 59DD2993
 P 6750 1350
-F 0 "C8" H 6775 1450 50  0000 L CNN
+F 0 "C3" H 6775 1450 50  0000 L CNN
 F 1 "1u" H 6775 1250 50  0000 L CNN
 F 2 "Capacitors_SMD:C_0805_HandSoldering" H 6788 1200 50  0001 C CNN
@@
 $EndComp
 $Comp
-L GND #PWR07
+L GND #PWR05
 U 1 1 59DD3DD1
 P 7100 1250
-F 0 "#PWR07" H 7100 1000 50  0001 C CNN
+F 0 "#PWR05" H 7100 1000 50  0001 C CNN
 F 1 "GND" H 7100 1100 50  0000 C CNN
 F 2 "" H 7100 1250 50  0001 C CNN
@@
 $EndComp
 $Comp
-L VCC #PWR08
+L VCC #PWR06
 U 1 1 59DD6B22
 P 7400 750
-F 0 "#PWR08" H 7400 600 50  0001 C CNN
+F 0 "#PWR06" H 7400 600 50  0001 C CNN
 F 1 "VCC" H 7400 900 50  0000 C CNN
 F 2 "" H 7400 750 50  0001 C CNN
@@
 $EndComp
 $Comp
-L VCC #PWR09
+L VCC #PWR07
 U 1 1 59DD6E46
 P 5550 850
-F 0 "#PWR09" H 5550 700 50  0001 C CNN
+F 0 "#PWR07" H 5550 700 50  0001 C CNN
 F 1 "VCC" H 5550 1000 50  0000 C CNN
 F 2 "" H 5550 850 50  0001 C CNN
@@
 $EndComp
 $Comp
-L VCC #PWR010
+L VCC #PWR08
 U 1 1 59DD796B
 P 3150 1150
-F 0 "#PWR010" H 3150 1000 50  0001 C CNN
+F 0 "#PWR08" H 3150 1000 50  0001 C CNN
 F 1 "VCC" H 3150 1300 50  0000 C CNN
 F 2 "" H 3150 1150 50  0001 C CNN
@@
 $EndComp
 $Comp
-L GND #PWR011
+L GND #PWR09
 U 1 1 59DD7D6F
 P 3100 1050
-F 0 "#PWR011" H 3100 800 50  0001 C CNN
+F 0 "#PWR09" H 3100 800 50  0001 C CNN
 F 1 "GND" H 3100 900 50  0000 C CNN
 F 2 "" H 3100 1050 50  0001 C CNN
@@
 NoConn ~ 3250 2350
 NoConn ~ 3250 2250
-NoConn ~ 3250 2150
 NoConn ~ 3250 1250
+$Comp
+L LED_ALT D13
+U 1 1 59E0695A
+P 2250 2150
+F 0 "D13" H 2250 2250 50  0000 C CNN
+F 1 "LED_ALT" H 2250 2050 50  0000 C CNN
+F 2 "LEDs:LED_0805_HandSoldering" H 2250 2150 50  0001 C CNN
+F 3 "" H 2250 2150 50  0001 C CNN
+	1    2250 2150
+	1    0    0    -1
+$EndComp
+$Comp
+L R R5
+U 1 1 59E08D67
+P 1900 2150
+F 0 "R5" V 1980 2150 50  0000 C CNN
+F 1 "10k" V 1900 2150 50  0000 C CNN
+F 2 "Resistors_SMD:R_0805_HandSoldering" V 1830 2150 50  0001 C CNN
+F 3 "" H 1900 2150 50  0001 C CNN
+	1    1900 2150
+	0    1    1    0
+$EndComp
+Wire Wire Line
+	2400 2150 3250 2150
+Wire Wire Line
+	2100 2150 2050 2150
+$Comp
+L GND #PWR010
+U 1 1 59E09893
+P 1700 2150
+F 0 "#PWR010" H 1700 1900 50  0001 C CNN
+F 1 "GND" H 1700 2000 50  0000 C CNN
+F 2 "" H 1700 2150 50  0001 C CNN
+F 3 "" H 1700 2150 50  0001 C CNN
+	1    1700 2150
+	0    1    1    0
+$EndComp
+Wire Wire Line
+	1750 2150 1700 2150
+Text Notes 4300 5150 0    60   ~ 0
+Shuttle\n
+Text Notes 7500 5300 0    60   ~ 0
+1
 $EndSCHEMATC
